Commit message: Add Gazebo simulation and ros2_control support

File: omnibot_description/urdf/mech/omni_wheel.urdf.xacro (robot description, xacro)
@@ -1,14 +1,15 @@
 <?xml version="1.0"?>
 <robot xmlns:xacro="http://www.ros.org/wiki/xacro">
+    <!-- TODO PARAMTERIZE MORE OF THE MEASUREMENTS -->
     <!-- Reusable wheel link and joint. Dimensions are placeholders until CAD is ready. -->
     <!-- This macro can be reused by putting using the line below in the base of the robot -->
-    <!-- <xacro:omni_wheel prefix="wheel_1" parent="base_link" x="${base_radius}" y="0.0" yaw="1.5708" /> -->
-    <xacro:macro name="omni_wheel" params="prefix parent x y yaw">
+    <!-- <xacro:omni_wheel suffix="wheel_1" parent="base_link" x="${base_radius}" y="0.0" yaw="1.5708" /> -->
+    <xacro:macro name="omni_wheel" params="suffix parent x y yaw">
         <xacro:property name="wheel_mass" value="0.5" />
         <xacro:property name="wheel_radius" value="0.1016" />
         <xacro:property name="wheel_length" value="0.0508" />
-        <joint name="${prefix}_joint" type="continuous">
+        <joint name="omni_wheel_joint_${suffix}" type="continuous">
             <parent link="${parent}" />
-            <child link="${prefix}_link" />
+            <child link="omni_wheel_link_${suffix}" />
             <!-- Defining center of the wheel's joint -->
             <origin xyz="${x} ${y} -.05" rpy="0 0 ${yaw}" />
@@ -16,5 +17,5 @@
             <axis xyz="0 1 0" />
         </joint>
-        <link name="${prefix}_link">
+        <link name="omni_wheel_link_${suffix}">
             <visual>
                 <!-- URDF cylinders use local Z as their length axis rotate it to align the axle with Y. -->

File: omnibot_description/urdf/mech/omnibot_base.urdf.xacro (robot description, xacro)
@@ -36,8 +36,8 @@
     </link>
     <!-- Three wheels spaced around the chassis. -->
-    <xacro:omni_wheel prefix="wheel_1" parent="base_link" x="${base_radius}" y="0.0" yaw="1.5708" />
-    <xacro:omni_wheel prefix="wheel_2" parent="base_link" x="${-base_radius / 2}"
+    <xacro:omni_wheel suffix="1" parent="base_link" x="${base_radius}" y="0.0" yaw="1.5708" />
+    <xacro:omni_wheel suffix="2" parent="base_link" x="${-base_radius / 2}"
         y="${base_radius * 0.866025}" yaw="3.6652" />
-    <xacro:omni_wheel prefix="wheel_3" parent="base_link" x="${-base_radius / 2}"
+    <xacro:omni_wheel suffix="3" parent="base_link" x="${-base_radius / 2}"
         y="${-base_radius * 0.866025}" yaw="-0.5236" />
 </robot>

File: omnibot_description/urdf/robots/omnibot.urdf.xacro (robot description, xacro)
@@ -10,7 +10,9 @@
   </material>
   <!-- Include statements to inject all of our URDF components -->
-  <xacro:include filename="../mech/inertials.urdf.xacro" />
-  <xacro:include filename="../mech/omnibot_base.urdf.xacro" />
-  <xacro:include filename="../sensors/lidar.urdf.xacro" />
-  <xacro:include filename="../sensors/camera.urdf.xacro" />
+  <xacro:include filename="$(find omnibot_description)/urdf/mech/inertials.urdf.xacro" />
+  <xacro:include filename="$(find omnibot_description)/urdf/mech/omnibot_base.urdf.xacro" />
+  <xacro:include filename="$(find omnibot_description)/urdf/sensors/lidar.urdf.xacro" />
+  <xacro:include filename="$(find omnibot_description)/urdf/sensors/camera.urdf.xacro" />
+  <xacro:include filename="$(find omnibot_description)/urdf/control/ros2_control.urdf.xacro" />
+  <xacro:include filename="$(find omnibot_description)/urdf/control/gazebo_plugin.urdf.xacro" />
 </robot>
