Commit message: Add simulated camera URDF and topic to Gazebo/ROS

File: omnibot_description/urdf/control/gazebo_plugin.urdf.xacro (robot description, xacro)
@@ -2,4 +2,5 @@
 <robot xmlns:xacro="http://ros.org/wiki/xacro">
     <gazebo>
+        <plugin filename="gz-sim-sensors-system" name="gz::sim::systems::Sensors" />
         <!-- Gazebo Control System Plugin -->
         <plugin filename="gz_ros2_control-system"

File: omnibot_description/urdf/mech/omnibot_base.urdf.xacro (robot description, xacro)
@@ -35,9 +35,10 @@
         </xacro:inertial_cylinder>
     </link>
-    <!-- Three wheels spaced around the chassis. -->
-    <xacro:omni_wheel suffix="1" parent="base_link" x="${base_radius}" y="0.0" yaw="1.5708" />
-    <xacro:omni_wheel suffix="2" parent="base_link" x="${-base_radius / 2}"
-        y="${base_radius * 0.866025}" yaw="3.6652" />
-    <xacro:omni_wheel suffix="3" parent="base_link" x="${-base_radius / 2}"
-        y="${-base_radius * 0.866025}" yaw="-0.5236" />
+    <!-- Three wheels spaced around the chassis -->
+    <xacro:omni_wheel suffix="1" parent="base_link" x="${base_radius / 2}"
+        y="${base_radius * 0.866025}" yaw="2.618" />
+    <xacro:omni_wheel suffix="2" parent="base_link" x="${base_radius / 2}"
+        y="${-base_radius * 0.866025}" yaw="0.524" />
+    <xacro:omni_wheel suffix="3" parent="base_link" x="-${base_radius}"
+        y="0.0" yaw="1.5708" />
 </robot>

File: omnibot_description/urdf/robots/omnibot.urdf.xacro (robot description, xacro)
@@ -4,8 +4,11 @@
   <!-- Global Color Definitions -->
   <material name="blue">
-    <color rgba="0.0 0.4 0.8 1.0"/>
+    <color rgba="0.0 0.4 0.8 1.0" />
+  </material>
+  <material name="red">
+    <color rgba="1.0 0.0 0.0 0.0" />
   </material>
   <material name="black">
-    <color rgba="0.0 0.0 0.0 1.0"/>
+    <color rgba="0.0 0.0 0.0 1.0" />
   </material>
   <!-- Include statements to inject all of our URDF components -->

File: omnibot_description/urdf/sensors/camera.urdf.xacro (robot description, xacro)
@@ -1,4 +1,50 @@
 <?xml version="1.0"?>
 <robot xmlns:xacro="http://www.ros.org/wiki/xacro">
-<!-- TODO -->
+    <joint name="camera_joint" type="fixed">
+        <parent link="base_link" />
+        <child link="camera_link" />
+        <origin xyz="0.385 0.05 0.03" rpy="0.0 0.0 0.0" />
+    </joint>
+    <link name="camera_link">
+        <visual>
+            <geometry>
+                <box size="0.05 0.03 0.03" />
+            </geometry>
+            <material name="red" />
+        </visual>
+    </link>
+     <!--Camera Optical Details:
+            This is added because we need to transform our coor system from
+            standard ROS orientation (x forward, y left, z up) to standard optical image
+            orientation (x right, y down, z forward(or away from camera))  -->
+    <joint name="camera_optical_joint" type="fixed">
+        <parent link="camera_link" />
+        <child link="camera_optical_link" />
+        <origin xyz="0 0 0" rpy="${-pi/2} 0 ${-pi/2}" />
+    </joint>
+    <link name="camera_optical_link"></link>
+    <!-- These tags actually make it so we can see what the gazebo entity sees on the camera topic. -->
+    <gazebo reference="camera_link">
+        <material>Gazebo/Red</material>
+        <sensor name="camera" type="camera">
+            <pose> 0 0 0 0 0 0</pose>
+            <visualize>true</visualize>
+            <update_rate>10</update_rate>
+            <camera>
+                <horizontal_fov>1.089</horizontal_fov>
+                <image>
+                    <format>R8G8B8</format>
+                    <width>640</width>
+                    <height>480</height>
+                </image>
+                <!-- Sees as close as .05 meters and as far as 8 meters -->
+                <clip>
+                    <near>0.05</near>
+                    <far>8.0</far>
+                </clip>
+            </camera>
+            <topic>camera/image_raw</topic>
+            <gz_frame_id>camera_link_optical</gz_frame_id>
+        </sensor>
+    </gazebo>
 </robot>
